File: CF_Interface_v2/cf_socket.kicad_sch (KiCad schematic)
At the start: 10 parts, among them J4 Socket_CF, U16 74HCT245, U17 74HCT245

Commit message: Modified CF_Interface card to use BERR and full AMx address modifier
These are some minor changes I made back in 2024 when I printed a copy
of the CF Interface card as part of the retroverse project.  The
original version didn't include all the address modifier pins from the
VME backplane, since the COMET uses a simplified version of VME, but
retroverse uses standard VME.  The change allows the card to ignore
incompatible cycles.

It's a bit messy, but I'm committing it as-is or I'll never get around
to it.
Parts:
- J4: footprint CF_Interface_v2:CF_Socket -> CF_Interface_v2:CF-Card_3M_N7E50-Q516RB-40
Changed lines of the file:
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@@
 				)
 				(justify left)
-				(hide yes)
 			)
 		)
@@
 				)
 				(justify right)
-				(hide yes)
 			)
 		)
@@
 				)
 				(justify right)
-				(hide yes)
 			)
 		)
@@
 				)
 				(justify right)
-				(hide yes)
 			)
 		)
@@
 				)
 				(justify right)
-				(hide yes)
 			)
 		)
@@
 				)
 				(justify left)
-				(hide yes)
 			)
 		)
@@
 				)
 				(justify left)
-				(hide yes)
 			)
 		)
@@
 				)
 				(justify right)
-				(hide yes)
 			)
 		)
@@
 				)
 				(justify right)
-				(hide yes)
 			)
 		)
@@
 				)
 				(justify right)
-				(hide yes)
 			)
 		)
@@
 				)
 				(justify left)
-				(hide yes)
 			)
 		)
@@
 				)
 				(justify right)
-				(hide yes)
 			)
 		)
@@
 			)
 		)
-		(property "Footprint" "CF_Interface_v2:CF_Socket"
+		(property "Footprint" "CF_Interface_v2:CF-Card_3M_N7E50-Q516RB-40"
 			(at 190.5 78.74 0)
 			(effects
